File: project/load_automatisation.kicad_pcb (KiCad board)
At the start: 2 copper layers, 76 x 88 mm, 33 parts, among them IC1 DRDC3105F-7, IC10 DRDC3105F-7, IC11 DRDC3105F-7, IC12 DRDC3105F-7, IC13 DRDC3105F-7, IC14 DRDC3105F-7, IC15 DRDC3105F-7, IC16 DRDC3105F-7, IC17 DRDC3105F-7, IC2 DRDC3105F-7, IC3 MC74VHC138DR2G, IC4 DRDC3105F-7, IC5 DRDC3105F-7, IC6 DRDC3105F-7, IC7 DRDC3105F-7, IC8 DRDC3105F-7, IC9 DRDC3105F-7, K1 IMC03TS, K10 IMC03TS, K11 IMC03TS, K12 IMC03TS, K13 IMC03TS, K14 IMC03TS, K15 IMC03TS, K16 IMC03TS, K2 V23079C1103B301, K3 V23079C1103B301, K4 V23079C1103B301, K5 V23079C1103B301, K6 V23079C1103B301, K7 V23079C1103B301, K8 V23079C1103B301, K9 V23079C1103B301

Commit message: first test
Parts:
- added DAQ: PinHeader_1x02_P2.54mm_Vertical, Connector_PinHeader_2.54mm:PinHeader_1x02_P2.54mm_Vertical, F.Cu at (112.0, 57.5)
- added R1: PinHeader_1x03_P2.54mm_Vertical, Connector_PinHeader_2.54mm:PinHeader_1x03_P2.54mm_Vertical, F.Cu at (112.5, 68.5)
- added R2: PinHeader_1x03_P2.54mm_Vertical, Connector_PinHeader_2.54mm:PinHeader_1x03_P2.54mm_Vertical, F.Cu at (112.5, 81.9)
- added R3: PinHeader_1x03_P2.54mm_Vertical, Connector_PinHeader_2.54mm:PinHeader_1x03_P2.54mm_Vertical, F.Cu at (112.5, 96.0)
- added R4: PinHeader_1x03_P2.54mm_Vertical, Connector_PinHeader_2.54mm:PinHeader_1x03_P2.54mm_Vertical, F.Cu at (73.0, 122.0)
- added R5: PinHeader_1x03_P2.54mm_Vertical, Connector_PinHeader_2.54mm:PinHeader_1x03_P2.54mm_Vertical, F.Cu at (43.5, 121.5)
- added R6: PinHeader_1x03_P2.54mm_Vertical, Connector_PinHeader_2.54mm:PinHeader_1x03_P2.54mm_Vertical, F.Cu at (67.0, 28.0)
- added R7: PinHeader_1x03_P2.54mm_Vertical, Connector_PinHeader_2.54mm:PinHeader_1x03_P2.54mm_Vertical, F.Cu at (24.0, 54.5)
- added R8: PinHeader_1x03_P2.54mm_Vertical, Connector_PinHeader_2.54mm:PinHeader_1x03_P2.54mm_Vertical, F.Cu at (24.5, 77.0)
- added TENG: PinHeader_1x02_P2.54mm_Vertical, Connector_PinHeader_2.54mm:PinHeader_1x02_P2.54mm_Vertical, F.Cu at (111.5, 48.0)
- added U1: AMS1117-5.0, Package_TO_SOT_SMD:SOT-223-3_TabPin2, F.Cu at (108.0, 38.5)
- added VCC: PinHeader_1x02_P2.54mm_Vertical, Connector_PinHeader_2.54mm:PinHeader_1x02_P2.54mm_Vertical, F.Cu at (118.0, 36.0)
Routing:
- net DAQ -: track 169.5 -> 242.3 mm
- net +5V: track 0.00 -> 51.4 mm
- net Rc_5: track 0.00 -> 33.8 mm
- net Rb_1: track 0.00 -> 33.0 mm
- net GND: track 213.8 -> 245.5 mm
- net Rb_2: track 0.00 -> 30.3 mm
- net Rb_5: track 0.00 -> 26.1 mm
- net Rc_4: track 0.00 -> 25.9 mm
- net Rc_1: track 0.00 -> 25.8 mm
- net Rb_3: track 0.00 -> 25.8 mm
- net Ra_1: track 0.00 -> 25.6 mm
- net Ra_2: track 0.00 -> 23.1 mm
- net Rc_2: track 0.00 -> 23.1 mm
- net Ra_8: track 0.00 -> 22.6 mm
- net Rc_7: track 0.00 -> 22.3 mm
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Other:
- board outline removed
